Commit message: Fix Rviz robot model

File: mini_mec_robot_gazebo.urdf (robot description, URDF)
Before this commit: robot wheeltec_robot, 8 links, 7 joints
Joints:
- joint lf_wheel_joint: axis 0 1 0 -> (none); type continuous -> fixed
- joint rf_wheel_joint: axis 0 1 0 -> (none); type continuous -> fixed
