Commit message: Switch simulation from Gazebo to Python 2D sim; fix stop and UI
Gazebo Classic and Ignition both crash (0xC0000139) on Windows ARM64 x64 emulation. Replace gzserver with Python 2D sim_node.py publishing /odom, /scan, /joint_states and TF odom->base_link. Add 0.5s cmd_vel timeout. Fix SimOutputWorker.stop() with taskkill /F /T. Rename Gazebo button to Simulate. Shrink RViz window to 1280x800. Add laser_link to mini_mec_robot.urdf.

Co-Authored-By: Claude Sonnet 4.6 <noreply@anthropic.com>

File: mini_mec_robot.urdf (robot description, URDF)
Before this commit: robot wheeltec_robot, 5 links, 4 joints
Links:
- added link laser_link; visual cylinder length=0.02 radius=0.03
Joints:
- added joint laser_joint: type fixed, parent base_link, child laser_link, origin xyz=0.0316 0.0001 0.0950 rpy=0 0 3.14159
